File: corne-cherry/pcb/corne-cherry.kicad_pcb (KiCad board)
At the start: 2 copper layers, 133.8 x 91.4 mm, 104 parts, among them J1 MJ-4PP-9, J2 OLED, J3 LED, P1 i2c-pin, P2 i2c-pin, SW1 SW_PUSH, SW10 SW_PUSH, SW11 SW_PUSH, SW12 SW_PUSH, SW13 SW_PUSH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

Commit message: Update readme and add PCB
Other:
- board text added: "Distux"
Changed lines of the file:
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@@
     (effects (font (size 0.7 0.7) (thickness 0.125)) (justify mirror))
+  )
+  (gr_text "Distux" (at 187.910724 99.523704) (layer "B.SilkS")
+    (effects (font (size 1.5 1.5) (thickness 0.3) bold) (justify left bottom mirror))
   )
   (gr_text "JLCJLCJLCJLC" (at 75.057 74.549) (layer "B.SilkS")
@@
     (effects (font (size 0.7 0.7) (thickness 0.125)))
   )
+  (gr_text "Distux" (at 182.190215 99.492615) (layer "F.SilkS")
+    (effects (font (size 1.5 1.5) (thickness 0.3) bold) (justify left bottom))
+  )
   (gr_text "Corne Cherry v2.2\nPCB designed by foostan\nEdit by Distux\n" (at 117.55 121.45) (layer "B.Mask")
